File: eurorack_balanced_out.sch (KiCad schematic (older format))
At the start: 31 parts, among them J1 Conn_01x02, J2 Conn_01x02, J3 Conn_02x05_Odd_Even, J4 AudioJack3, J5 AudioJack3, U1 THAT1646W16, U2 THAT1646W16

Commit message: reannotate
Parts:
- gave numbers to parts that had none: 4

Commit message: fix weird erc non connected error
Connections:
- wire segments 137 -> 139
Changed lines of the file:
@@
 Wire Wire Line
 	6200 5350 6200 5450
-Wire Wire Line
-	6000 5050 5900 5050
-Wire Wire Line
-	5600 5050 5500 5050
-Wire Wire Line
-	5500 5050 5500 4300
-Wire Wire Line
-	5900 5050 5900 4100
 $Comp
 L power:GND #PWR0101
@@
 Connection ~ 5300 4300
 Wire Wire Line
-	5300 4300 6250 4300
+	5300 4300 5500 4300
 Wire Wire Line
 	5200 4100 5300 4100
@@
 Connection ~ 5300 4100
 Wire Wire Line
-	5300 4100 6250 4100
+	5300 4100 5900 4100
 Wire Wire Line
 	3900 6050 3900 6000
@@
 	0    1    1    0
 $EndComp
+Wire Wire Line
+	5600 5050 5500 5050
+Wire Wire Line
+	6000 5050 5900 5050
+Wire Wire Line
+	5500 5050 5500 4300
+Connection ~ 5500 4300
+Wire Wire Line
+	5500 4300 6250 4300
+Wire Wire Line
+	5900 5050 5900 4100
+Connection ~ 5900 4100
+Wire Wire Line
+	5900 4100 6250 4100
 $EndSCHEMATC

Commit message: fix power connector footprint
Parts:
- J3: footprint Connector_PinHeader_2.54mm:PinHeader_2x04_P2.54mm_Vertical -> Connector_PinHeader_2.54mm:PinHeader_2x05_P2.54mm_Vertical
Changed lines of the file:
@@
 F 0 "J3" H 3500 6800 50  0000 C CNN
 F 1 "Conn_02x05_Odd_Even" H 2950 6800 50  0000 C CNN
-F 2 "Connector_PinHeader_2.54mm:PinHeader_2x04_P2.54mm_Vertical" H 3200 6300 50  0001 C CNN
+F 2 "Connector_PinHeader_2.54mm:PinHeader_2x05_P2.54mm_Vertical" H 3200 6300 50  0001 C CNN
 F 3 "~" H 3200 6300 50  0001 C CNN
 	1    3200 6300

Commit message: add some mouser part numbers
Parts:
- C10, C11, C12, C9: Mouser 80-C0805C101JAGAUTO -> 80-C0805C101JAGAUTO
- C3, C4: Mouser 80-C0805C104K5RACLR -> 80-C0805C104K5RACLR
- D1, D2, D3, D4: Mouser (none) -> 863-BAV99LT1G
- FB1, FB2, FB3, FB4: Mouser 81-BLM21A601F -> 81-BLM21A601F
Changed lines of the file:
@@
 F 2 "Capacitor_SMD:C_0805_2012Metric_Pad1.15x1.40mm_HandSolder" H 4388 6000 50  0001 C CNN
 F 3 "~" H 4350 6150 50  0001 C CNN
-F 4 " 80-C0805C104K5RACLR" V 4350 6150 50  0001 C CNN "Mouser"
+F 4 "80-C0805C104K5RACLR" V 4350 6150 50  0001 C CNN "Mouser"
 	1    4350 6150
 	-1   0    0    1
@@
 F 2 "Capacitor_SMD:C_0805_2012Metric_Pad1.15x1.40mm_HandSolder" H 4388 6300 50  0001 C CNN
 F 3 "~" H 4350 6450 50  0001 C CNN
-F 4 " 80-C0805C104K5RACLR" V 4350 6450 50  0001 C CNN "Mouser"
+F 4 "80-C0805C104K5RACLR" V 4350 6450 50  0001 C CNN "Mouser"
 	1    4350 6450
 	-1   0    0    1
@@
 F 2 "Resistor_SMD:R_0805_2012Metric_Pad1.15x1.40mm_HandSolder" V 6280 1600 50  0001 C CNN
 F 3 "~" H 6350 1600 50  0001 C CNN
-F 4 " 81-BLM21A601F" V 6350 1600 50  0001 C CNN "Mouser"
+F 4 "81-BLM21A601F" V 6350 1600 50  0001 C CNN "Mouser"
 	1    6350 1600
 	0    1    1    0
@@
 F 2 "Capacitor_SMD:C_0805_2012Metric_Pad1.15x1.40mm_HandSolder" H 6500 1950 50  0001 C CNN
 F 3 "~" H 6500 1950 50  0001 C CNN
-F 4 " 80-C0805C101JAGAUTO " H 6500 1950 50  0001 C CNN "Mouser"
+F 4 "80-C0805C101JAGAUTO " H 6500 1950 50  0001 C CNN "Mouser"
 	1    6500 1950
 	1    0    0    -1
@@
 F 2 "Resistor_SMD:R_0805_2012Metric_Pad1.15x1.40mm_HandSolder" V 6280 1800 50  0001 C CNN
 F 3 "~" H 6350 1800 50  0001 C CNN
-F 4 " 81-BLM21A601F" V 6350 1800 50  0001 C CNN "Mouser"
+F 4 "81-BLM21A601F" V 6350 1800 50  0001 C CNN "Mouser"
 	1    6350 1800
 	0    1    1    0
@@
 F 2 "Capacitor_SMD:C_0805_2012Metric_Pad1.15x1.40mm_HandSolder" H 6850 1950 50  0001 C CNN
 F 3 "~" H 6850 1950 50  0001 C CNN
-F 4 " 80-C0805C101JAGAUTO " H 6850 1950 50  0001 C CNN "Mouser"
+F 4 "80-C0805C101JAGAUTO " H 6850 1950 50  0001 C CNN "Mouser"
 	1    6850 1950
 	1    0    0    -1
@@
 F 2 "Resistor_SMD:R_0805_2012Metric_Pad1.15x1.40mm_HandSolder" V 6280 4100 50  0001 C CNN
 F 3 "~" H 6350 4100 50  0001 C CNN
-F 4 " 81-BLM21A601F" V 6350 4100 50  0001 C CNN "Mouser"
+F 4 "81-BLM21A601F" V 6350 4100 50  0001 C CNN "Mouser"
 	1    6350 4100
 	0    1    1    0
@@
 F 2 "Capacitor_SMD:C_0805_2012Metric_Pad1.15x1.40mm_HandSolder" H 6500 4450 50  0001 C CNN
 F 3 "~" H 6500 4450 50  0001 C CNN
-F 4 " 80-C0805C101JAGAUTO " H 6500 4450 50  0001 C CNN "Mouser"
+F 4 "80-C0805C101JAGAUTO " H 6500 4450 50  0001 C CNN "Mouser"
 	1    6500 4450
 	1    0    0    -1
@@
 F 2 "Resistor_SMD:R_0805_2012Metric_Pad1.15x1.40mm_HandSolder" V 6280 4300 50  0001 C CNN
 F 3 "~" H 6350 4300 50  0001 C CNN
-F 4 " 81-BLM21A601F" V 6350 4300 50  0001 C CNN "Mouser"
+F 4 "81-BLM21A601F" V 6350 4300 50  0001 C CNN "Mouser"
 	1    6350 4300
 	0    1    1    0
@@
 F 2 "Capacitor_SMD:C_0805_2012Metric_Pad1.15x1.40mm_HandSolder" H 6850 4450 50  0001 C CNN
 F 3 "~" H 6850 4450 50  0001 C CNN
-F 4 " 80-C0805C101JAGAUTO " H 6850 4450 50  0001 C CNN "Mouser"
+F 4 "80-C0805C101JAGAUTO " H 6850 4450 50  0001 C CNN "Mouser"
 	1    6850 4450
 	1    0    0    -1
@@
 F 2 "Package_TO_SOT_SMD:SOT-23" H 5800 2050 50  0001 C CNN
 F 3 "https://assets.nexperia.com/documents/data-sheet/BAV99_SER.pdf" H 5800 2550 50  0001 C CNN
+F 4 "863-BAV99LT1G" H 5800 2550 50  0001 C CNN "Mouser"
 	1    5800 2550
 	0    1    -1   0
@@
 F 2 "Package_TO_SOT_SMD:SOT-23" H 6200 2050 50  0001 C CNN
 F 3 "https://assets.nexperia.com/documents/data-sheet/BAV99_SER.pdf" H 6200 2550 50  0001 C CNN
+F 4 "863-BAV99LT1G" H 6200 2550 50  0001 C CNN "Mouser"
 	1    6200 2550
 	0    1    -1   0
@@
 F 2 "Package_TO_SOT_SMD:SOT-23" H 5800 4550 50  0001 C CNN
 F 3 "https://assets.nexperia.com/documents/data-sheet/BAV99_SER.pdf" H 5800 5050 50  0001 C CNN
+F 4 "863-BAV99LT1G" H 5800 5050 50  0001 C CNN "Mouser"
 	1    5800 5050
 	0    1    -1   0
@@
 F 2 "Package_TO_SOT_SMD:SOT-23" H 6200 4550 50  0001 C CNN
 F 3 "https://assets.nexperia.com/documents/data-sheet/BAV99_SER.pdf" H 6200 5050 50  0001 C CNN
+F 4 "863-BAV99LT1G" H 6200 5050 50  0001 C CNN "Mouser"
 	1    6200 5050
 	0    1    -1   0

Commit message: fix some resistor values
Parts:
- R3, R4: value 3.9k -> 1.2k
Changed lines of the file:
@@
 P 3750 1750
 F 0 "R3" H 3691 1704 50  0000 R CNN
-F 1 "3.9k" H 3691 1795 50  0000 R CNN
+F 1 "1.2k" H 3691 1795 50  0000 R CNN
 F 2 "Resistor_SMD:R_0805_2012Metric_Pad1.15x1.40mm_HandSolder" H 3750 1750 50  0001 C CNN
 F 3 "~" H 3750 1750 50  0001 C CNN
@@
 P 3750 4250
 F 0 "R4" H 3691 4204 50  0000 R CNN
-F 1 "3.9k" H 3691 4295 50  0000 R CNN
+F 1 "1.2k" H 3691 4295 50  0000 R CNN
 F 2 "Resistor_SMD:R_0805_2012Metric_Pad1.15x1.40mm_HandSolder" H 3750 4250 50  0001 C CNN
 F 3 "~" H 3750 4250 50  0001 C CNN

Commit message: finish mouser part numbers
Parts:
- J1, J2: Mouser (none) -> 200-TSW10207TS
- J3: Mouser (none) -> 200-TSS10501TD
- J4, J5: Mouser (none) -> 568-NJ3FD-V
- R1, R2: Mouser (none) -> 667-ERJ-6ENF3901V
- R3, R4: Mouser (none) -> 667-ERJ-S06F1201V
- U1, U2: Mouser (none) -> 887-1646W16-U
Changed lines of the file:
@@
 F 2 "Package_SO:SOIC-16W_7.5x10.3mm_P1.27mm" H 4750 2050 50  0001 C CNN
 F 3 "http://www.thatcorp.com/datashts/THAT_1606-1646_Datasheet.pdf" H 4750 2050 50  0001 C CNN
+F 4 "887-1646W16-U" H 4900 1700 50  0001 C CNN "Mouser"
 	1    4900 1700
 	1    0    0    -1
@@
 F 2 "Connector_PinHeader_2.54mm:PinHeader_2x05_P2.54mm_Vertical" H 3200 6300 50  0001 C CNN
 F 3 "~" H 3200 6300 50  0001 C CNN
+F 4 "200-TSS10501TD" H 3200 6300 50  0001 C CNN "Mouser"
 	1    3200 6300
 	1    0    0    -1
@@
 F 2 "Connector_PinHeader_2.54mm:PinHeader_1x02_P2.54mm_Vertical" H 3050 1600 50  0001 C CNN
 F 3 "~" H 3050 1600 50  0001 C CNN
+F 4 "200-TSW10207TS" H 3050 1600 50  0001 C CNN "Mouser"
 	1    3050 1600
 	-1   0    0    -1
@@
 F 2 "Connector_Audio:Jack_6.35mm_Neutrik_NJ3FD-V_Vertical" H 7650 1700 50  0001 C CNN
 F 3 "~" H 7650 1700 50  0001 C CNN
+F 4 "568-NJ3FD-V" H 7650 1700 50  0001 C CNN "Mouser"
 	1    7650 1700
 	-1   0    0    1
@@
 F 2 "Package_SO:SOIC-16W_7.5x10.3mm_P1.27mm" H 4750 4550 50  0001 C CNN
 F 3 "http://www.thatcorp.com/datashts/THAT_1606-1646_Datasheet.pdf" H 4750 4550 50  0001 C CNN
+F 4 "887-1646W16-U" H 4900 4200 50  0001 C CNN "Mouser"
 	1    4900 4200
 	1    0    0    -1
@@
 F 2 "Connector_PinHeader_2.54mm:PinHeader_1x02_P2.54mm_Vertical" H 3050 4100 50  0001 C CNN
 F 3 "~" H 3050 4100 50  0001 C CNN
+F 4 "200-TSW10207TS" H 3050 4100 50  0001 C CNN "Mouser"
 	1    3050 4100
 	-1   0    0    -1
@@
 F 2 "Connector_Audio:Jack_6.35mm_Neutrik_NJ3FD-V_Vertical" H 7650 4200 50  0001 C CNN
 F 3 "~" H 7650 4200 50  0001 C CNN
+F 4 "568-NJ3FD-V" H 7650 4200 50  0001 C CNN "Mouser"
 	1    7650 4200
 	-1   0    0    1
@@
 F 2 "Resistor_SMD:R_0805_2012Metric_Pad1.15x1.40mm_HandSolder" H 3750 1750 50  0001 C CNN
 F 3 "~" H 3750 1750 50  0001 C CNN
+F 4 "667-ERJ-S06F1201V" H 3750 1750 50  0001 C CNN "Mouser"
 	1    3750 1750
 	-1   0    0    1
@@
 F 2 "Resistor_SMD:R_0805_2012Metric_Pad1.15x1.40mm_HandSolder" H 3600 1600 50  0001 C CNN
 F 3 "~" H 3600 1600 50  0001 C CNN
+F 4 "667-ERJ-6ENF3901V" H 3600 1600 50  0001 C CNN "Mouser"
 	1    3600 1600
 	0    1    1    0
@@
 F 2 "Resistor_SMD:R_0805_2012Metric_Pad1.15x1.40mm_HandSolder" H 3750 4250 50  0001 C CNN
 F 3 "~" H 3750 4250 50  0001 C CNN
+F 4 "667-ERJ-S06F1201V" H 3750 4250 50  0001 C CNN "Mouser"
 	1    3750 4250
 	-1   0    0    1
@@
 F 2 "Resistor_SMD:R_0805_2012Metric_Pad1.15x1.40mm_HandSolder" H 3600 4100 50  0001 C CNN
 F 3 "~" H 3600 4100 50  0001 C CNN
+F 4 "667-ERJ-6ENF3901V" H 3600 4100 50  0001 C CNN "Mouser"
 	1    3600 4100
 	0    1    1    0

Commit message: use different footprint for 10uF cap so we can use the 25V version
Parts:
- C5, C6, C7, C8: footprint Capacitor_SMD:CP_Elec_5x5.4 -> Capacitor_SMD:CP_Elec_6.3x5.4
Changed lines of the file:
@@
 F 0 "C5" V 4871 1350 50  0000 C CNN
 F 1 "10u" V 4962 1350 50  0000 C CNN
-F 2 "Capacitor_SMD:CP_Elec_5x5.4" H 5100 1350 50  0001 C CNN
+F 2 "Capacitor_SMD:CP_Elec_6.3x5.4" H 5100 1350 50  0001 C CNN
 F 3 "~" H 5100 1350 50  0001 C CNN
 F 4 "647-UWP1C100MCL" V 5100 1350 50  0001 C CNN "Mouser"
@@
 F 0 "C7" V 4871 3850 50  0000 C CNN
 F 1 "10u" V 4962 3850 50  0000 C CNN
-F 2 "Capacitor_SMD:CP_Elec_5x5.4" H 5100 3850 50  0001 C CNN
+F 2 "Capacitor_SMD:CP_Elec_6.3x5.4" H 5100 3850 50  0001 C CNN
 F 3 "~" H 5100 3850 50  0001 C CNN
 F 4 "647-UWP1C100MCL" V 5100 3850 50  0001 C CNN "Mouser"
@@
 F 0 "C8" V 4871 4550 50  0000 C CNN
 F 1 "10u" V 4962 4550 50  0000 C CNN
-F 2 "Capacitor_SMD:CP_Elec_5x5.4" H 5100 4550 50  0001 C CNN
+F 2 "Capacitor_SMD:CP_Elec_6.3x5.4" H 5100 4550 50  0001 C CNN
 F 3 "~" H 5100 4550 50  0001 C CNN
 F 4 "647-UWP1C100MCL" V 5100 4550 50  0001 C CNN "Mouser"
@@
 F 0 "C6" V 5300 2050 50  0000 C CNN
 F 1 "10u" V 5200 2050 50  0000 C CNN
-F 2 "Capacitor_SMD:CP_Elec_5x5.4" H 5100 2050 50  0001 C CNN
+F 2 "Capacitor_SMD:CP_Elec_6.3x5.4" H 5100 2050 50  0001 C CNN
 F 3 "~" H 5100 2050 50  0001 C CNN
 F 4 "647-UWP1C100MCL" V 5100 2050 50  0001 C CNN "Mouser"

Commit message: change mouser part number for 10u non polarized caps to 25v version
Parts:
- C5, C6, C7, C8: Mouser 647-UWP1C100MCL -> 647-UWP1E100MCL
Changed lines of the file:
@@
 F 2 "Capacitor_SMD:CP_Elec_6.3x5.4" H 5100 1350 50  0001 C CNN
 F 3 "~" H 5100 1350 50  0001 C CNN
-F 4 "647-UWP1C100MCL" V 5100 1350 50  0001 C CNN "Mouser"
+F 4 "647-UWP1E100MCL" V 5100 1350 50  0001 C CNN "Mouser"
 	1    5100 1350
 	0    1    1    0
@@
 F 2 "Capacitor_SMD:CP_Elec_6.3x5.4" H 5100 3850 50  0001 C CNN
 F 3 "~" H 5100 3850 50  0001 C CNN
-F 4 "647-UWP1C100MCL" V 5100 3850 50  0001 C CNN "Mouser"
+F 4 "647-UWP1E100MCL" V 5100 3850 50  0001 C CNN "Mouser"
 	1    5100 3850
 	0    1    1    0
@@
 F 2 "Capacitor_SMD:CP_Elec_6.3x5.4" H 5100 4550 50  0001 C CNN
 F 3 "~" H 5100 4550 50  0001 C CNN
-F 4 "647-UWP1C100MCL" V 5100 4550 50  0001 C CNN "Mouser"
+F 4 "647-UWP1E100MCL" V 5100 4550 50  0001 C CNN "Mouser"
 	1    5100 4550
 	0    1    1    0
@@
 F 2 "Capacitor_SMD:CP_Elec_6.3x5.4" H 5100 2050 50  0001 C CNN
 F 3 "~" H 5100 2050 50  0001 C CNN
-F 4 "647-UWP1C100MCL" V 5100 2050 50  0001 C CNN "Mouser"
+F 4 "647-UWP1E100MCL" V 5100 2050 50  0001 C CNN "Mouser"
 	1    5100 2050
 	0    1    1    0
